File: SolderStation/SolderStation.sch (KiCad schematic (older format))
At the start: 0 parts

Commit message: Revert "Add files via upload"
This reverts commit 9e82852e4677a33747f2b205dd1fce6c4e717f3a.
Changed lines of the file:
@@
 LIBS:contrib
 LIBS:valves
+LIBS:Remus
 LIBS:SolderStation-cache
 EELAYER 25 0
@@
 F1 "PowerSupply.sch" 60
 F2 "24VAC" O R 3800 3750 60
-F3 "5VDC" O R 3800 3000 60
-F4 "12VDC" O R 3800 2900 60
+F4 "12VDC" O R 3800 3000 60
 F5 "EARTH" O R 3800 4200 60
 F6 "GNDDC" O R 3800 3200 60
 F7 "GNDAC" O R 3800 3900 60
 F8 "3.3VDC" O R 3800 3100 60
+F9 "PG" O R 3800 2850 60
 $EndSheet
 $Sheet
@@
 F10 "Ch3_Temp" O R 6050 4000 60
 F11 "3.3VDC" I L 4250 3100 60
+F12 "CH1_PWM" I R 6050 3100 60
+F13 "CH2_PWM" I R 6050 3200 60
+F14 "CH3_PWM" I R 6050 3300 60
+F15 "+12V" I L 4250 3000 60
 $EndSheet
 $Sheet
@@
 F0 "Control" 60
 F1 "Control.sch" 60
-F2 "PWM_Ch1" O L 6500 2800 60
-F3 "PWM_Ch2" O L 6500 3250 60
-F4 "PWM_Ch3" O L 6500 3700 60
-F5 "TC+_Ch1" I L 6500 2900 60
-F6 "TC-_Ch1" I L 6500 3000 60
-F7 "TC+_Ch2" I L 6500 3350 60
-F8 "TC-_Ch2" I L 6500 3450 60
-F9 "TC+_Ch3" I L 6500 3800 60
-F10 "TC-_Ch3" I L 6500 3900 60
+F2 "Ch1_PWM" O L 6500 3100 60
+F3 "Ch2_PWM" O L 6500 3200 60
+F4 "Ch3_PWM" O L 6500 3300 60
+F5 "PG" I L 6500 2800 60
+F6 "~CS~" O L 6500 3700 60
+F7 "CLK" O L 6500 3600 60
+F8 "Ch1_TEMP" I L 6500 3800 60
+F9 "Ch2_TEMP" I L 6500 3900 60
+F10 "Ch3_TEMP" I L 6500 4000 60
+F11 "3V3" I L 6500 2900 60
+F12 "GND" I L 6500 3000 60
 $EndSheet
 Wire Wire Line
@@
 	3800 4200 4250 4200
 Wire Wire Line
-	4250 3100 3800 3100
+	3800 3100 4250 3100
 Wire Wire Line
 	3800 3200 4250 3200
+Wire Wire Line
+	3800 2850 4000 2850
+Wire Wire Line
+	4000 2850 4000 2500
+Wire Wire Line
+	4000 2500 6300 2500
+Wire Wire Line
+	6500 3100 6050 3100
+Wire Wire Line
+	6050 3200 6500 3200
+Wire Wire Line
+	6500 3300 6050 3300
+Wire Wire Line
+	6500 3600 6050 3600
+Wire Wire Line
+	6050 3700 6500 3700
+Wire Wire Line
+	6500 4000 6050 4000
+Wire Wire Line
+	6050 3900 6500 3900
+Wire Wire Line
+	6500 3800 6050 3800
+Wire Wire Line
+	6500 3000 6100 3000
+Wire Wire Line
+	6100 3000 6100 2600
+Wire Wire Line
+	6100 2600 4200 2600
+Wire Wire Line
+	4100 2550 6200 2550
+Wire Wire Line
+	6200 2550 6200 2900
+Wire Wire Line
+	6200 2900 6500 2900
+Wire Wire Line
+	6500 2800 6300 2800
+Wire Wire Line
+	6300 2800 6300 2500
+Wire Wire Line
+	4200 2600 4200 3200
+Connection ~ 4200 3200
+Wire Wire Line
+	4100 2550 4100 3100
+Connection ~ 4100 3100
+Wire Wire Line
+	3800 3000 4250 3000
 $EndSCHEMATC
